Commit message: added new urdf

File: urdf/abb.urdf (robot description, URDF)
Before this commit: robot irb120, 11 links, 10 joints
Links:
- link base_link: geometry collision mesh filename=file:///home/omar-magdy/gp_ws/install/ros2srrc_robots/share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; visual mesh filename=file:///home/omar-magdy/gp_ws/install/ros2srrc_robots/share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
- link link_1: geometry collision mesh filename=file:///home/omar-magdy/gp_ws/install/ros2srrc_robots/share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; visual mesh filename=file:///home/omar-magdy/gp_ws/install/ros2srrc_robots/share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
- link link_2: geometry collision mesh filename=file:///home/omar-magdy/gp_ws/install/ros2srrc_robots/share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; visual mesh filename=file:///home/omar-magdy/gp_ws/install/ros2srrc_robots/share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
- link link_3: geometry collision mesh filename=file:///home/omar-magdy/gp_ws/install/ros2srrc_robots/share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; visual mesh filename=file:///home/omar-magdy/gp_ws/install/ros2srrc_robots/share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
- link link_4: geometry collision mesh filename=file:///home/omar-magdy/gp_ws/install/ros2srrc_robots/share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; visual mesh filename=file:///home/omar-magdy/gp_ws/install/ros2srrc_robots/share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
- link link_5: geometry collision mesh filename=file:///home/omar-magdy/gp_ws/install/ros2srrc_robots/share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; visual mesh filename=file:///home/omar-magdy/gp_ws/install/ros2srrc_robots/share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
- link link_6: geometry collision mesh filename=file:///home/omar-magdy/gp_ws/install/ros2srrc_robots/share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; visual mesh filename=file:///home/omar-magdy/gp_ws/install/ros2srrc_robots/share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

File: urdf/ar4.urdf (robot description, URDF)
Before this commit: robot ar4, 12 links, 11 joints
Links:
- link ar4_base_link: geometry collision mesh filename=file:///home/omar-magdy/gp_ws/install/annin_ar4_description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; visual mesh filename=file:///home/omar-magdy/gp_ws/install/annin_ar4_description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
- link ar4_gripper_base_link: geometry collision mesh filename=file:///home/omar-magdy/gp_ws/install/annin_ar4_description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; visual mesh filename=file:///home/omar-magdy/gp_ws/install/annin_ar4_description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
- link ar4_gripper_jaw1_link: geometry collision mesh filename=file:///home/omar-magdy/gp_ws/install/annin_ar4_description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; visual mesh filename=file:///home/omar-magdy/gp_ws/install/annin_ar4_description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
- link ar4_gripper_jaw2_link: geometry collision mesh filename=file:///home/omar-magdy/gp_ws/install/annin_ar4_description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; visual mesh filename=file:///home/omar-magdy/gp_ws/install/annin_ar4_description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
- link ar4_link_1: geometry collision mesh filename=file:///home/omar-magdy/gp_ws/install/annin_ar4_description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; visual mesh filename=file:///home/omar-magdy/gp_ws/install/annin_ar4_description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
- link ar4_link_2: geometry collision mesh filename=file:///home/omar-magdy/gp_ws/install/annin_ar4_description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; visual mesh filename=file:///home/omar-magdy/gp_ws/install/annin_ar4_description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
- link ar4_link_3: geometry collision mesh filename=file:///home/omar-magdy/gp_ws/install/annin_ar4_description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; visual mesh filename=file:///home/omar-magdy/gp_ws/install/annin_ar4_description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
- link ar4_link_4: geometry collision mesh filename=file:///home/omar-magdy/gp_ws/install/annin_ar4_description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; visual mesh filename=file:///home/omar-magdy/gp_ws/install/annin_ar4_description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
- link ar4_link_5: geometry collision mesh filename=file:///home/omar-magdy/gp_ws/install/annin_ar4_description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; visual mesh filename=file:///home/omar-magdy/gp_ws/install/annin_ar4_description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
- link ar4_link_6: geometry collision mesh filename=file:///home/omar-magdy/gp_ws/install/annin_ar4_description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; visual mesh filename=file:///home/omar-magdy/gp_ws/install/annin_ar4_description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

File: urdf/dual_arms.urdf (robot description, URDF)
Before this commit: robot dual_arms, 22 links, 21 joints
Links:
- removed link world
- link ar4_base_link: geometry collision mesh filename=file:///home/omar-magdy/gp_ws/install/annin_ar4_description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; visual mesh filename=file:///home/omar-magdy/gp_ws/install/annin_ar4_description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
- link ar4_gripper_base_link: geometry collision mesh filename=file:///home/omar-magdy/gp_ws/install/annin_ar4_description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; visual mesh filename=file:///home/omar-magdy/gp_ws/install/annin_ar4_description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
- link ar4_gripper_jaw1_link: geometry collision mesh filename=file:///home/omar-magdy/gp_ws/install/annin_ar4_description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; visual mesh filename=file:///home/omar-magdy/gp_ws/install/annin_ar4_description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
- link ar4_gripper_jaw2_link: geometry collision mesh filename=file:///home/omar-magdy/gp_ws/install/annin_ar4_description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; visual mesh filename=file:///home/omar-magdy/gp_ws/install/annin_ar4_description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
- link ar4_link_1: geometry collision mesh filename=file:///home/omar-magdy/gp_ws/install/annin_ar4_description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; visual mesh filename=file:///home/omar-magdy/gp_ws/install/annin_ar4_description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
- link ar4_link_2: geometry collision mesh filename=file:///home/omar-magdy/gp_ws/install/annin_ar4_description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; visual mesh filename=file:///home/omar-magdy/gp_ws/install/annin_ar4_description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
- link ar4_link_3: geometry collision mesh filename=file:///home/omar-magdy/gp_ws/install/annin_ar4_description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; visual mesh filename=file:///home/omar-magdy/gp_ws/install/annin_ar4_description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
- link ar4_link_4: geometry collision mesh filename=file:///home/omar-magdy/gp_ws/install/annin_ar4_description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; visual mesh filename=file:///home/omar-magdy/gp_ws/install/annin_ar4_description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
- link ar4_link_5: geometry collision mesh filename=file:///home/omar-magdy/gp_ws/install/annin_ar4_description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; visual mesh filename=file:///home/omar-magdy/gp_ws/install/annin_ar4_description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
- link ar4_link_6: geometry collision mesh filename=file:///home/omar-magdy/gp_ws/install/annin_ar4_description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; visual mesh filename=file:///home/omar-magdy/gp_ws/install/annin_ar4_description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
- link base_link: geometry collision mesh filename=file:///home/omar-magdy/gp_ws/install/ros2srrc_robots/share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; visual mesh filename=file:///home/omar-magdy/gp_ws/install/ros2srrc_robots/share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
- link link_1: geometry collision mesh filename=file:///home/omar-magdy/gp_ws/install/ros2srrc_robots/share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; visual mesh filename=file:///home/omar-magdy/gp_ws/install/ros2srrc_robots/share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
- link link_2: geometry collision mesh filename=file:///home/omar-magdy/gp_ws/install/ros2srrc_robots/share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; visual mesh filename=file:///home/omar-magdy/gp_ws/install/ros2srrc_robots/share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
- link link_3: geometry collision mesh filename=file:///home/omar-magdy/gp_ws/install/ros2srrc_robots/share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; visual mesh filename=file:///home/omar-magdy/gp_ws/install/ros2srrc_robots/share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
- link link_4: geometry collision mesh filename=file:///home/omar-magdy/gp_ws/install/ros2srrc_robots/share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; visual mesh filename=file:///home/omar-magdy/gp_ws/install/ros2srrc_robots/share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
- link link_5: geometry collision mesh filename=file:///home/omar-magdy/gp_ws/install/ros2srrc_robots/share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; visual mesh filename=file:///home/omar-magdy/gp_ws/install/ros2srrc_robots/share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
- link link_6: geometry collision mesh filename=file:///home/omar-magdy/gp_ws/install/ros2srrc_robots/share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; visual mesh filename=file:///home/omar-magdy/gp_ws/install/ros2srrc_robots/share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
Joints:
- removed joint ar4_base_joint
- removed joint irb120_world_joint

File: urdf/dual_arms.urdf.xacro (robot description, xacro)
@@ -20,13 +20,4 @@
     <xacro:include filename="$(find ros2srrc_hmi)/urdf/hmicamera.urdf.xacro"/>
   </xacro:if>
-  <!-- World -->
-  <link name="world"/>
-  <!-- 🔹 AR4 Robot -->
-  <xacro:ar_robot
-    tf_prefix="$(arg tf_prefix)"
-    parent="world"
-    robot_parameters_file="$(find annin_ar4_description)/config/$(arg ar_model).yaml">
-    <origin xyz="0 0 0" rpy="0 0 -1.57"/>
-  </xacro:ar_robot>
   <!-- AR4 Gripper -->
   <xacro:if value="$(arg include_gripper)">
@@ -41,10 +32,4 @@
     EE="$(arg EE)"
     EE_name="$(arg EE_name)"/>
-  <!-- IRB120 Fixed Joint to World with offset -->
-  <joint name="irb120_world_joint" type="fixed">
-    <parent link="world"/>
-    <child link="base_link"/>
-    <origin xyz="-1.2 0 0" rpy="0 0 0"/>
-  </joint>
   <!-- Optional: HMI Camera -->
   <xacro:if value="$(arg hmi)">

File: urdf/stand.urdf.xacro (robot description, xacro)
@@ -24,5 +24,5 @@
       <geometry>
         <mesh
-          filename="file:///home/mariamelsebaey/gp_ws/src/dual_arms/meshes/base_link.STL" />
+          filename="file:///home/omar-magdy/gp_ws/src/dual_arms/meshes/base_link.STL" />
       </geometry>
       <material
@@ -38,5 +38,5 @@
       <geometry>
         <mesh
-          filename="file:///home/mariamelsebaey/gp_ws/src/dual_arms/meshes/base_link.STL" />
+          filename="file:///home/omar-magdy/gp_ws/src/dual_arms/meshes/base_link.STL" />
       </geometry>
     </collision>
